Commit message: Add camera config to sim

File: sim/scenes/sensors.xacro (robot description, xacro)
@@ -1,6 +1,7 @@
 <?xml version="1.0"?>
 <robot xmlns:xacro="http://www.ros.org/wiki/xacro">
-  <xacro:property name="cam_res_width" default="352"/>
-  <xacro:property name="cam_res_height" default="240"/>
+  <xacro:property name="cam_res_width" default="1288"/>
+  <xacro:property name="cam_res_height" default="964"/>
+  <xacro:property name="cam_fov" default = "109"/>
   <!-- angle defines position, vert defines whether it's vertical (1) or horizontal (0), orientation is angle it's facing (0 if vert) -->
   <xacro:macro name="camera" params="name down">
@@ -20,4 +21,5 @@
         <y>0</y>
       </orientation>
+      <fovy> ${cam_fov} </fovy>
     </virtualCamera>
   </xacro:macro>
