Commit message: Fixed an issue with the buoy path

File: sim/scenes/GateScene.xml.xacro (robot description, xacro)
@@ -98,7 +98,7 @@
     </orientation>
   </vehicle>
-  <!-- <vehicle>
+ <vehicle>
    <name> buoy </name>
-   <file>sim/scenes/meshes/buoy.urdf</file>
+   <file>$(find sim)/scenes/buoy.urdf</file>
    <position>
      <x> 0</x>
@@ -116,5 +116,5 @@
      <z> .5 </z>
    </scaleFactor>
-</vehicle> -->
+</vehicle>
   <object>
     <name>terrain</name>

File: sim/scenes/buoy.urdf (robot description, URDF)
Before this commit: robot Buoy, 1 links, 0 joints
Links:
- link red_buoy: mass None -> 20
