Commit message: UUV initial integration

File: core/descriptions/alfie_description/urdf/base.xacro (robot description, xacro)
@@ -35,5 +35,5 @@
         </inertial>
         <visual>
-          <origin xyz="0 0 0" rpy="0 0 0"/>
+          <origin xyz="0 0 0" rpy="${pi} 0 0"/>
           <geometry>
             <mesh filename="${visual_mesh_file}" scale="1 1 1" />
@@ -41,5 +41,5 @@
         </visual>
         <collision>
-          <origin xyz="0 0 0" rpy="${pi} 0 0"/>
+          <origin xyz="0 0 0" rpy="0 0 0"/>
           <geometry>
             <mesh filename="${collision_mesh_file}" scale="1 1 1" />

File: core/descriptions/alfie_description/urdf/gazebo.xacro (robot description, xacro)
@@ -2,5 +2,5 @@
 <robot xmlns:xacro="http://www.ros.org/wiki/xacro">
     <!-- Center of buoyancy -->
-    <xacro:property name="alfie_cob" value="0 0 0.1"/>
+    <xacro:property name="alfie_cob" value="0 0 -0.1"/>
     <!-- Vehicle's actual volume (Gazebo cannot compute the volume out of the mesh) -->
     <xacro:property name="alfie_volume" value=".021"/>
