Commit message: leaving

File: core/descriptions/alfie_description/urdf/actuators.xacro (robot description, xacro)
@@ -8,5 +8,5 @@
           aware that Gazebo does not use the SNAME convention per default.
     -->
-    <xacro:thruster_macro robot_namespace="${namespace}" thruster_id="0">
+    <!-- <xacro:thruster_macro robot_namespace="${namespace}" thruster_id="0">
         <origin xyz="0 0 0" rpy="0 0 ${pi}" />
     </xacro:thruster_macro>
@@ -16,4 +16,4 @@
     <xacro:thruster_macro robot_namespace="${namespace}" thruster_id="2">
     <origin xyz="0 0 0" rpy="0 -${0.5*pi} 0" />
-    </xacro:thruster_macro>
+    </xacro:thruster_macro> -->
 </robot>

File: core/descriptions/alfie_description/urdf/base.xacro (robot description, xacro)
@@ -50,11 +50,4 @@
       <selfCollide>false</selfCollide>
     </gazebo>
-    <underwater_dynamics>
-      <buoyancy value="21"/>
-      <center_of_buoyancy x="0" y = "0" z = "0.1" />
-      <added_mass x="0" y="0" z="0" k="0" m="0" n="0" />
-      <linear_damping_coeffs x="0" y="0" z="0" k="0" m="0" n="0" />
-      <rate value="50" />
-    </underwater_dynamics>
     <!-- Set up hydrodynamic plugin given as input parameter -->
     <xacro:insert_block name="gazebo"/>

File: core/descriptions/alfie_description/urdf/gazebo.xacro (robot description, xacro)
@@ -4,8 +4,8 @@
     <xacro:property name="alfie_cob" value="0 0 0.1"/>
     <!-- Vehicle's actual volume (Gazebo cannot compute the volume out of the mesh) -->
-    <xacro:property name="alfie_volume" value="21"/>
+    <xacro:property name="alfie_volume" value=".021"/>
     <!-- Describing the dimensions of the vehicle's bounding box -->
-    <xacro:property name="alfie_length" value=".5"/>
-    <xacro:property name="alfie_width"  value=".5"/>
+    <xacro:property name="alfie_length" value=".25"/>
+    <xacro:property name="alfie_width"  value=".25"/>
     <xacro:property name="alfie_height" value=".25"/>
     <xacro:macro name="alfie_hydro_model" params="namespace">
@@ -13,5 +13,5 @@
       <link name="${namespace}/base_link">
         <!-- This flag will make the link neutrally buoyant -->
-        <neutrally_buoyant>1</neutrally_buoyant>
+        <neutrally_buoyant>0</neutrally_buoyant>
         <!-- Link's volume -->
         <volume>${alfie_volume}</volume>
@@ -49,5 +49,5 @@
           -->
           <linear_damping>
-            0 0 0 0 0 0
+            -10 -10 -10 -10 -10 -10
           </linear_damping>
           <!--
@@ -89,8 +89,8 @@
         <!-- 2) This computes the added-mass and damping parameters for a sphere
         in the fluid with the given radius -->
-        <hydrodynamic_model>
+        <!-- <hydrodynamic_model>
           <type>sphere</type>
-          <radius>.25</radius>
-        </hydrodynamic_model>
+          <radius>.5</radius>
+        </hydrodynamic_model> -->
       </link>
     </xacro:macro>

Commit message: Dynamics for sim w./ thruster alloc

File: core/descriptions/alfie_description/urdf/actuators.xacro (robot description, xacro)
@@ -8,12 +8,35 @@
           aware that Gazebo does not use the SNAME convention per default.
     -->
-    <!-- <xacro:thruster_macro robot_namespace="${namespace}" thruster_id="0">
-        <origin xyz="0 0 0" rpy="0 0 ${pi}" />
+    <!-- Horizontal Front Left -->
+    <xacro:thruster_macro robot_namespace="${namespace}" thruster_id="0">
+        <origin xyz=".277 -.277 -.049" rpy="0 0 ${pi/4}" />
     </xacro:thruster_macro>
+    <!-- Horizontal Front Right -->
     <xacro:thruster_macro robot_namespace="${namespace}" thruster_id="1">
-        <origin xyz="0 0 0" rpy="0 0 ${pi}" />
+        <origin xyz=".277 .277 -.049" rpy="0 0 ${-1*pi/4}" />
     </xacro:thruster_macro>
+    <!-- Horizontal Back Left -->
     <xacro:thruster_macro robot_namespace="${namespace}" thruster_id="2">
-    <origin xyz="0 0 0" rpy="0 -${0.5*pi} 0" />
-    </xacro:thruster_macro> -->
+        <origin xyz="-.277 -.277 -.049" rpy="0 0 ${-1*pi/4}" />
+    </xacro:thruster_macro>
+    <!-- Horizontal Back Right -->
+    <xacro:thruster_macro robot_namespace="${namespace}" thruster_id="3">
+        <origin xyz="-.277 .277 -.049" rpy="0 0 ${pi/4}" />
+    </xacro:thruster_macro>
+    <!-- Vertical Front Left -->
+    <xacro:thruster_macro robot_namespace="${namespace}" thruster_id="4">
+        <origin xyz=".121 -.279 .054" rpy="0 ${pi/2} 0" />
+    </xacro:thruster_macro>
+    <!-- Vertical Front Right -->
+    <xacro:thruster_macro robot_namespace="${namespace}" thruster_id="5">
+        <origin xyz=".121 .279 .054" rpy="0 ${pi/2} 0" />
+    </xacro:thruster_macro>
+    <!-- Vertical Back Left -->
+    <xacro:thruster_macro robot_namespace="${namespace}" thruster_id="6">
+        <origin xyz="-.121 -.279 .054" rpy="0 ${pi/2} 0" />
+    </xacro:thruster_macro>
+    <!-- Vertical Back Right -->
+    <xacro:thruster_macro robot_namespace="${namespace}" thruster_id="7">
+        <origin xyz="-.121 .279 .054" rpy="0 ${pi/2} 0" />
+    </xacro:thruster_macro>
 </robot>

File: core/descriptions/alfie_description/urdf/snippets.xacro (robot description, xacro)
@@ -78,36 +78,4 @@
           <type>ZeroOrder</type>
         </dynamics>
-        <!-- 2) First order model -->
-        <dynamics>
-          <type>FirstOrder</type>
-          <timeConstant>0.0</timeConstant>
-        </dynamics>
-        <!-- 3) Yoerger's nonlinear dynamic model
-        For information on the model description:
-        [1] D. R. Yoerger, J. G. Cooke, and J.-J. E. Slotine, "The influence of
-            thruster dynamics on underwater vehicle behavior and their incorporation
-            into control system design," IEEE Journal of Oceanic Engineering, vol. 15,
-            no. 3, pp. 167-178, Jul. 1990.
-        -->
-        <dynamics>
-          <type>Yoerger</type>
-          <alpha>0.0</alpha>
-          <beta>0.0</beta>
-        </dynamics>
-        <!-- 4) Bessa's nonlinear dynamic model
-        For information on the model description:
-        [2] Bessa, Wallace Moreira, Max Suell Dutra, and Edwin Kreuzer. "Thruster
-            dynamics compensation for the positioning of underwater robotic vehicles
-            through a fuzzy sliding mode based approach." ABCM Symposium Series in
-            Mechatronics. Vol. 2. 2006.
-        -->
-        <dynamics>
-          <type>Bessa</type>
-          <Jmsp>0.0</Jmsp>
-          <Kv1>0.0</Kv1>
-          <Kv2>0.0</Kv2>
-          <Kt>0.0</Kt>
-          <Rm>0.0</Rm>
-        </dynamics>
         <!--
         Choose one of the model for the steady-state curve describing the
@@ -121,5 +89,5 @@
         <conversion>
           <type>Basic</type>
-          <rotorConstant>0.0</rotorConstant>
+          <rotorConstant>0.01</rotorConstant>
         </conversion>
         <!-- 2) Dead-zone nonlinearity described in Bessa, 2006
@@ -130,5 +98,4 @@
         thrust = 0, if deltaL < x * abs(x) < deltaR
         thrust = rotorConstantR * (x * abs(x) - deltaR), if x * abs(x) >= deltaL
-        -->
         <conversion>
           <type>Bessa</type>
@@ -138,10 +105,9 @@
           <deltaR>0.0</deltaR>
         </conversion>
-        <!-- 3) Linear interpolation
+        3) Linear interpolation
         If you have access to the thruster's data sheet, for example,
         you can enter samples of the curve's input and output values
         and the thruster output will be found through linear interpolation
         of the given samples.
-        -->
         <conversion>
           <type>LinearInterp</type>
@@ -149,4 +115,5 @@
           <outputValues>0 1 2 3</outputValues>
         </conversion>
+      -->
       </plugin>
     </gazebo>
