Commit message: thruster allocation working

File: core/descriptions/alfie_description/urdf/actuators_accurate_z.xacro (robot description, xacro)
@@ -10,33 +10,33 @@
     <!-- Horizontal Front Left -->
     <xacro:thruster_macro robot_namespace="${namespace}" thruster_id="0">
-        <origin xyz=".277 -.277 0.0" rpy="0 0 ${pi/4}" />
+        <origin xyz=".277 -.277 -.049" rpy="0 0 ${pi/4}" />
     </xacro:thruster_macro>
     <!-- Horizontal Front Right -->
     <xacro:thruster_macro robot_namespace="${namespace}" thruster_id="1">
-        <origin xyz=".277 .277 0.0" rpy="0 0 ${-1*pi/4}" />
+        <origin xyz=".277 .277 -.049" rpy="0 0 ${-1*pi/4}" />
     </xacro:thruster_macro>
     <!-- Horizontal Back Left -->
     <xacro:thruster_macro robot_namespace="${namespace}" thruster_id="2">
-        <origin xyz="-.277 -.277 0.0" rpy="0 0 ${3*pi/4}" />
+        <origin xyz="-.277 -.277 -.049" rpy="0 0 ${-1*pi/4}" />
     </xacro:thruster_macro>
     <!-- Horizontal Back Right -->
     <xacro:thruster_macro robot_namespace="${namespace}" thruster_id="3">
-        <origin xyz="-.277 .277 0.0" rpy="0 0 ${-3*pi/4}" />
+        <origin xyz="-.277 .277 -.049" rpy="0 0 ${pi/4}" />
     </xacro:thruster_macro>
     <!-- Vertical Front Left -->
     <xacro:thruster_macro robot_namespace="${namespace}" thruster_id="4">
-        <origin xyz=".121 -.279 0.0" rpy="0 ${pi/2} 0" />
+        <origin xyz=".121 -.279 .054" rpy="0 ${pi/2} 0" />
     </xacro:thruster_macro>
     <!-- Vertical Front Right -->
     <xacro:thruster_macro robot_namespace="${namespace}" thruster_id="5">
-        <origin xyz=".121 .279 0.0" rpy="0 ${pi/2} 0" />
+        <origin xyz=".121 .279 .054" rpy="0 ${pi/2} 0" />
     </xacro:thruster_macro>
     <!-- Vertical Back Left -->
     <xacro:thruster_macro robot_namespace="${namespace}" thruster_id="6">
-        <origin xyz="-.121 -.279 0.0" rpy="0 ${pi/2} 0" />
+        <origin xyz="-.121 -.279 .054" rpy="0 ${pi/2} 0" />
     </xacro:thruster_macro>
     <!-- Vertical Back Right -->
     <xacro:thruster_macro robot_namespace="${namespace}" thruster_id="7">
-        <origin xyz="-.121 .279 0.0" rpy="0 ${pi/2} 0" />
+        <origin xyz="-.121 .279 .054" rpy="0 ${pi/2} 0" />
     </xacro:thruster_macro>
 </robot>

File: core/descriptions/alfie_description/urdf/snippets.xacro (robot description, xacro)
@@ -89,5 +89,5 @@
         <conversion>
           <type>Basic</type>
-          <rotorConstant>0.01</rotorConstant>
+          <rotorConstant>1</rotorConstant>
         </conversion>
         <!-- 2) Dead-zone nonlinearity described in Bessa, 2006
