Commit message: Dynamics simulation tentatively working

File: core/descriptions/alfie_description/robots/default.urdf (robot description, URDF)
Before this commit: robot alfie, 1 links, 0 joints
Links:
- added link alfie/dvl_link; collision cylinder length=1e-06 radius=1e-06; visual mesh filename=file:///home/sethgi/catkin_ws/src/MuddSub/sim/plugins/meshe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 scale=1 1 1
- added link alfie/dvl_sonar0_link, mass 0.001; collision cylinder length=1e-06 radius=1e-06
- added link alfie/dvl_sonar1_link, mass 0.001; collision cylinder length=1e-06 radius=1e-06
- added link alfie/dvl_sonar2_link, mass 0.001; collision cylinder length=1e-06 radius=1e-06
- added link alfie/dvl_sonar3_link, mass 0.001; collision cylinder length=1e-06 radius=1e-06
Joints:
- added joint alfie/dvl_joint: type revolute, parent alfie/base_link, child alfie/dvl_link, origin xyz=0 0 0 rpy=0 0 0, axis 1 0 0, limit lower=0 upper=0 effort=0 velocity=0
- added joint alfie/dvl_sonar0_joint: type revolute, parent alfie/dvl_link, child alfie/dvl_sonar0_link, origin xyz=0 0 0 rpy=0 -0.52 0.0, axis 1 0 0, limit lower=0 upper=0 effort=0 velocity=0
- added joint alfie/dvl_sonar1_joint: type revolute, parent alfie/dvl_link, child alfie/dvl_sonar1_link, origin xyz=0 0 0 rpy=0 0 0.52, axis 1 0 0, limit lower=0 upper=0 effort=0 velocity=0
- added joint alfie/dvl_sonar2_joint: type revolute, parent alfie/dvl_link, child alfie/dvl_sonar2_link, origin xyz=0 0 0 rpy=0 0.52 0.0, axis 1 0 0, limit lower=0 upper=0 effort=0 velocity=0
- added joint alfie/dvl_sonar3_joint: type revolute, parent alfie/dvl_link, child alfie/dvl_sonar3_link, origin xyz=0 0 0 rpy=0 0.0 -0.52, axis 1 0 0, limit lower=0 upper=0 effort=0 velocity=0

File: core/descriptions/alfie_description/urdf/base.xacro (robot description, xacro)
@@ -9,4 +9,6 @@
   <!-- Loading vehicle's specific macros -->
   <xacro:include filename="$(find core)/descriptions/alfie_description/urdf/snippets.xacro"/>
+  <!-- DVL A50 -->
+  <xacro:include filename="$(find sim)/plugins/urdf/dvl.xacro" />
   <!--
     Vehicle's parameters (remember to enter the model parameters below)

File: core/descriptions/alfie_description/urdf/sensors.xacro (robot description, xacro)
@@ -8,7 +8,13 @@
   -->
   <!-- DVL  -->
-  <!-- <xacro:default_dvl namespace="${namespace}" parent_link="${namespace}/base_link">
-    <origin xyz="-.163 0 .0375" rpy="0 0 0"/>
-  </xacro:default_dvl> -->
+  <xacro:dvl_a50 namespace="${namespace}" parent_link="${namespace}/base_link"
+    suffix=""
+    reference_frame="world_ned"
+    update_rate="7"
+    topic="dvl"
+    noise_sigma="0"
+    noise_amplitude="0">
+    <origin xyz=".1 0 0.00635" rpy="${pi} 0 0" />
+  </xacro:dvl_a50>
   <!-- Mount a camera  -->
   <!-- <xacro:default_camera namespace="${namespace}" parent_link="${namespace}/base_link" suffix="">
