Commit message: fastslam appears to work

File: core/descriptions/alfie.urdf.xacro (robot description, xacro)
@@ -11,7 +11,7 @@
     <visual>
       <origin rpy="${pi} 0 0" xyz="0 0 0"/>
-      <geometry>
+      <!-- <geometry>
         <mesh filename="$(find core)/descriptions/meshes/AlfieVisual.STL"/>
-      </geometry>
+      </geometry> -->
     </visual>
     <underwater_dynamics>

File: sim/scenes/GateScene.xml.xacro (robot description, xacro)
@@ -47,5 +47,5 @@
     </offsetr>
   </simParams>
-  <camera>
+  <!-- <camera>
     <freeMotion> 1 </freeMotion>
     <objectToTrack>Alfie/base_link</objectToTrack>
@@ -64,5 +64,5 @@
       <z>0 </z>
     </lookAt>
-  </camera>
+  </camera> -->
   <vehicle>
     <name>Alfie</name>

Commit message: Setup obstacles and Alfie in sim

File: core/descriptions/alfie.urdf.xacro (robot description, xacro)
@@ -11,7 +11,7 @@
     <visual>
       <origin rpy="${pi} 0 0" xyz="0 0 0"/>
-      <!-- <geometry>
+      <geometry>
         <mesh filename="$(find core)/descriptions/meshes/AlfieVisual.STL"/>
-      </geometry> -->
+      </geometry>
     </visual>
     <underwater_dynamics>

File: sim/scenes/GateScene.xml.xacro (robot description, xacro)
@@ -69,12 +69,12 @@
     <file>$(find core)/descriptions/alfie.urdf</file>
     <position>
-      <x> 0</x>
-      <y> 0 </y>
-      <z> 0 </z>
-    </position>
-    <orientation>
-      <r>0</r>
-      <p>0</p>
-      <y>-1.57</y>
+      <x> 0 </x>
+      <y> 0 </y>
+      <z> 1 </z>
+    </position>
+    <orientation>
+      <r>0</r>
+      <p>0</p>
+      <y>0</y>
     </orientation>
     <xacro:include filename="$(find sim)/scenes/sensors.xacro" />
@@ -98,5 +98,5 @@
     </orientation>
   </vehicle>
- <vehicle>
+ <!-- <vehicle>
    <name> buoy </name>
    <file>$(find sim)/scenes/buoy.urdf</file>
@@ -125,5 +125,5 @@
     <y>0</y>
   </orientation>
-</vehicle>
+</vehicle> -->
   <object>
     <name>terrain</name>
